File: Input/Poti/Poti.sch (EAGLE design)
At the start: 5 parts

Commit message: sort out
Parts:
- removed U$4: MVS0608, thar:MVS0608
- added U$3: POTI3382G, thar:POTI3382G
- U$1: value CARRIER_SMD2SMD2_3POL -> CARRIER_SMD2SMD2_3POL_W; device thar:CARRIER_SMD2SMD2_3POL -> thar:CARRIER_SMD2SMD2_3POL_W
Connections:
- removed net N$5: U$10.4, U$4.0
- net GND: now also U$3.A
- net N$2: now also U$10.5, U$3.S; no longer U$10.3, U$4.1
- net VCC: now also U$3.E
Changed lines of the file:
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@@
 <parts>
 <part name="FRAME1" library="frames" deviceset="A5L-LOC" device=""/>
-<part name="U$1" library="thar" deviceset="CARRIER_SMD2" device="SMD2_3POL" value="CARRIER_SMD2SMD2_3POL"/>
+<part name="U$1" library="thar" deviceset="CARRIER_SMD2" device="SMD2_3POL_W" value="CARRIER_SMD2SMD2_3POL_W"/>
 <part name="P+3" library="supply1" deviceset="VCC" device=""/>
 <part name="GND3" library="supply1" deviceset="GND" device=""/>
@@
 <part name="GND5" library="supply1" deviceset="GND" device=""/>
 <part name="GND6" library="supply1" deviceset="GND" device=""/>
-<part name="U$4" library="thar" deviceset="MVS0608" device=""/>
+<part name="P+1" library="supply1" deviceset="VCC" device=""/>
 <part name="GND2" library="supply1" deviceset="GND" device=""/>
-<part name="P+1" library="supply1" deviceset="VCC" device=""/>
+<part name="U$3" library="thar" deviceset="POTI" device="3382G"/>
+<part name="P+2" library="supply1" deviceset="VCC" device=""/>
+<part name="GND4" library="supply1" deviceset="GND" device=""/>
 </parts>
 <sheets>
@@
 <instance part="GND5" gate="1" x="129.54" y="114.3"/>
 <instance part="GND6" gate="1" x="71.12" y="96.52"/>
-<instance part="U$4" gate="A" x="48.26" y="111.76" rot="R180"/>
+<instance part="P+1" gate="VCC" x="152.4" y="106.68"/>
 <instance part="GND2" gate="1" x="144.78" y="104.14"/>
-<instance part="P+1" gate="VCC" x="152.4" y="106.68"/>
+<instance part="U$3" gate="G$1" x="43.18" y="91.44"/>
+<instance part="P+2" gate="VCC" x="40.64" y="99.06"/>
+<instance part="GND4" gate="1" x="40.64" y="83.82"/>
 </instances>
 <busses>
@@
 <wire x1="144.78" y1="106.68" x2="157.48" y2="106.68" width="0.1524" layer="91"/>
 </segment>
+<segment>
+<pinref part="U$3" gate="G$1" pin="A"/>
+<pinref part="GND4" gate="1" pin="GND"/>
+</segment>
 </net>
 <net name="VCC" class="0">
@@
 <wire x1="152.4" y1="104.14" x2="157.48" y2="104.14" width="0.1524" layer="91"/>
 </segment>
+<segment>
+<pinref part="U$3" gate="G$1" pin="E"/>
+<pinref part="P+2" gate="VCC" pin="VCC"/>
+</segment>
 </net>
 <net name="N$2" class="0">
 <segment>
-<pinref part="U$10" gate="G$1" pin="3"/>
-<pinref part="U$4" gate="A" pin="1"/>
-<wire x1="76.2" y1="111.76" x2="58.42" y2="111.76" width="0.1524" layer="91"/>
+<pinref part="U$3" gate="G$1" pin="S"/>
+<pinref part="U$10" gate="G$1" pin="5"/>
+<wire x1="45.72" y1="91.44" x2="76.2" y2="106.68" width="0.1524" layer="91"/>
 </segment>
 </net>
-<net name="N$5" class="0">
-<segment>
-<pinref part="U$10" gate="G$1" pin="4"/>
-<pinref part="U$4" gate="A" pin="0"/>
-<wire x1="76.2" y1="109.22" x2="58.42" y2="109.22" width="0.1524" layer="91"/>
-</segment>
-</net>
